File: supply.sch (KiCad schematic (older format))
At the start: 115 parts, among them IC1 TPS54561, IC2 NCP380HMUAJAATBG, J3 DC_SOCKET, Q1 BC817W, U10 REF3012AIDBZT, U11 AP2303MPTR-G1, U7 INA199A1DCKR, U8 INA199A1DCKR, U9 DA9062-00AM1-BA

Commit message: Add title block to the schematic sheets and some TODOs
Connections:
- wire segments 281 -> 280
Other:
- note added: "TODO: consider switching into Ti LPDDR PMIC"
Changed lines of the file:
@@
 $Descr A3 16535 11693
 encoding utf-8
-Sheet 5 8
-Title ""
+Sheet 6 8
+Title "LPDDR4 Test Board"
 Date ""
-Rev ""
+Rev "1.0.0"
 Comp ""
 Comment1 ""
@@
 	14325 7900 14125 7900
 Wire Wire Line
-	12600 7800 12700 7800
-Connection ~ 12600 7800
-Wire Wire Line
-	12375 7800 12600 7800
-Wire Wire Line
 	12600 8200 13075 8200
 Wire Wire Line
@@
 	0    1    1    0
 $EndComp
+Wire Wire Line
+	12375 7800 12700 7800
+Text Notes 12425 4975 0    59   ~ 12
+TODO: consider switching into Ti LPDDR PMIC
 $EndSCHEMATC

Commit message: Add preliminary PMIC
Parts:
- removed C134, C135, C137, C138, C140, C146, C147: C_2u2_0402, lpddr4-test-board-footprints:0402-cap, symbol lpddr4-test-board:C_2u2_0402
- removed C136: C_10n_0402, lpddr4-test-board-footprints:0402-cap, symbol lpddr4-test-board:C_10n_0402
- removed C139, C141, C144, C145: C_22u_0805_10V, lpddr4-test-board-footprints:0805-cap, symbol lpddr4-test-board:C_22u_0805_10V
- removed C142, C143, C149, C150, C173: C_100n_0402_6V3, lpddr4-test-board-footprints:0402-cap, symbol lpddr4-test-board:C_100n_0402_6V3
- removed C148: C_470n_0402, lpddr4-test-board-footprints:0402-cap, symbol lpddr4-test-board:C_470n_0402
- removed C151, C152, C154, C155, C156, C157, C159, C160, C181: C_47u_0603, lpddr4-test-board-footprints:0603-cap, symbol lpddr4-test-board:C_47u_0603
- removed C168, C179: C_10u_0402, lpddr4-test-board-footprints:0402-cap, symbol lpddr4-test-board:C_10u_0402
- removed C176: C_1u_0402, lpddr4-test-board-footprints:0402-cap, symbol lpddr4-test-board:C_1u_0402
- removed L1, L2, L3, L4: 1uH, lpddr4-test-board-footprints:SRP2512A-1R0M, symbol lpddr4-test-board:1uH
- removed Q1: BC817W, lpddr4-test-board-footprints:SOT-323, symbol lpddr4-test-board:BC817W-antmicroTransistorsBipolarSingle
- removed R100: R_4k99_0402, lpddr4-test-board-footprints:0402-res, symbol lpddr4-test-board:R_4k99_0402
- removed R101, R104, R112, R113, R121: R_1k_0402, lpddr4-test-board-footprints:0402-res, symbol lpddr4-test-board:R_1k_0402
- removed R102: R_825R_0402, lpddr4-test-board-footprints:0402-res, symbol lpddr4-test-board:R_825R_0402
- removed R103: R_15k_0603, lpddr4-test-board-footprints:0603-res, symbol lpddr4-test-board:R_15k_0603
- removed R105: R_931R_0402, lpddr4-test-board-footprints:0402-res, symbol lpddr4-test-board:R_931R_0402
- removed R106: R_200k_0402, lpddr4-test-board-footprints:0402-res, symbol lpddr4-test-board:R_200k_0402
- removed R107, R84, R85, R86, R87, R95, R96: R_10k_0402, lpddr4-test-board-footprints:0402-res, symbol lpddr4-test-board:R_10k_0402
- removed R108, R109, R110, R117, R94, R97, R98: R_0R_0402, lpddr4-test-board-footprints:0402-res, symbol lpddr4-test-board:R_0R_0402
- removed R111: R_0R01_1206, lpddr4-test-board-footprints:1206-res, symbol lpddr4-test-board:R_0R01_1206
- removed R88, R90: R_6k34_0402, lpddr4-test-board-footprints:0402-res, symbol lpddr4-test-board:R_6k34_0402
- removed R89, R91: R_100R_0402, lpddr4-test-board-footprints:0402-res, symbol lpddr4-test-board:R_100R_0402
- removed R92, R93, R99: R_100k_0402, lpddr4-test-board-footprints:0402-res, symbol lpddr4-test-board:R_100k_0402
- removed U11: AP2303MPTR-G1, lpddr4-test-board-footprints:SOIC127P600X172-8N, symbol lpddr4-test-board:AP2303MPTR-G1
- removed U7, U8: INA199A1DCKR, lpddr4-test-board-footprints:SOT-SC70-6, symbol lpddr4-test-board:INA199A1DCKR
- removed U9: DA9062-00AM1-BA, lpddr4-test-board-footprints:DA9062-00AM1-BA, symbol lpddr4-test-board:DA9062-00AM1-BA
- added C? (x3): C_10u_0402, lpddr4-test-board-footprints:0402-cap, symbol lpddr4-test-board:C_10u_0402
- added C? (x2): C_100n_0402_6V3, lpddr4-test-board-footprints:0402-cap, symbol lpddr4-test-board:C_100n_0402_6V3
- added C?: C_1u_0402, lpddr4-test-board-footprints:0402-cap, symbol lpddr4-test-board:C_1u_0402
- added C? (x6): C_22u_0603, lpddr4-test-board-footprints:0603-cap, symbol lpddr4-test-board:C_22u_0603
- added C?: C_470n_0402, lpddr4-test-board-footprints:0402-cap, symbol lpddr4-test-board:C_470n_0402
- added C? (x3): C_10u_25V_0603, lpddr4-test-board-footprints:0603-cap, symbol lpddr4-test-board:C_10u_25V_0603
- added C?: C_10u_0603, lpddr4-test-board-footprints:0603-cap, symbol lpddr4-test-board:C_10u_0603
- added C?: C_100n_0402_16V, lpddr4-test-board-footprints:0402-cap, symbol lpddr4-test-board:C_100n_0402_16V
- added C?: C_2u2_0402, lpddr4-test-board-footprints:0402-cap, symbol lpddr4-test-board:C_2u2_0402
- added C?: C_100p_0402, lpddr4-test-board-footprints:0402-cap, symbol lpddr4-test-board:C_100p_0402
- added L?: IHLP1212AEERR47M11, lpddr4-test-board-footprints:IHLP-1212AE, symbol lpddr4-test-board:IHLP1212AEERR47M11
- added L?: IHLP2020BZER4R7M01, lpddr4-test-board-footprints:IHLP2020BZER4R7M01, symbol lpddr4-test-board:IHLP2020BZER4R7M01
- added L?: DFE322512F-R68M=P2, lpddr4-test-board-footprints:INDC3225X120N, symbol lpddr4-test-board:DFE322512F-R68M=P2
- added Q?: BC817W, lpddr4-test-board-footprints:SOT-323, symbol lpddr4-test-board:BC817W
- added R?: R_100k_0402, lpddr4-test-board-footprints:0402-res, symbol lpddr4-test-board:R_100k_0402
- added R?: R_5R1_1020, lpddr4-test-board-footprints:1020-res, symbol lpddr4-test-board:R_5R1_1020
- added R?: R_0R_0402, lpddr4-test-board-footprints:0402-res, symbol lpddr4-test-board:R_0R_0402
- added R?: R_243k_0402, lpddr4-test-board-footprints:0402-res, symbol lpddr4-test-board:R_243k_0402
- added R?: R_53k6_0402, lpddr4-test-board-footprints:0402-res, symbol lpddr4-test-board:R_53k6_0402
- added U?: TPS65296, lpddr4-test-board-footprints:VQFN-HR, symbol lpddr4-test-board:TPS65296
- added U?: TPS62823DLCT, lpddr4-test-board-footprints:QFN-8_2x1mm, symbol lpddr4-test-board:TPS62823DLCT
Connections:
- net labels added: VDD0V6, VDD1V1, VDD1V8, VDDEN, VDDQEN
- net labels removed: DDRVCC, DDRVREF, DDRVTT, GPIO2, GPIO3, GPIO4, PMIC_SCL, PMIC_SDA, SNS5V0+, SNS5V0-, SNS5V0_N, SNS5V0_P, SNSVCCINT+, SNSVCCINT-, SNSVCCINT_N, SNSVCCINT_P, VBUCK1, VBUCK2, VBUCK3, VBUCK4, VCC1V8, VCC_INT, VSN5V0+, VSNS5V0+, VSNS5V0-, VSNS5V0_N, VSNS5V0_P, VSNSVU_N, VSNSVU_P
- wire segments 280 -> 151
- no-connect marks 4 -> 1
Other:
- note added: "3V3 supply (1A)"
- note added: "TODO: check if VDD labels have the same names as those connected to FPGA"
- note added: "TODO: check whether this part of the design is obsolete"
- note added: "VCC5V0 4.5V to 5.5V"
- note added: "VDD1V1 0.6V 1.5A"
- note added: "VDD1V1 1.1V 8A"
- note added: "VDD1V8 1.8V 1A"
- note added: "VIN 4.5V to 18V"
- note removed: "10V"
- note removed: "Current sense"
- note removed: "DDR PMIC (1.75A)"
- note removed: "TODO: consider switching into Ti LPDDR PMIC"
- moved on the sheet: C153, C158, C161, C162, C163, C164, C165, C166, C167, C169, C170, C171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

Commit message: Update supply related circuits
Parts:
- removed R125: R_0R005_1206, lpddr4-test-board-footprints:1206-res, symbol lpddr4-test-board:R_0R005_1206
- added R? (x5): R_0R_1206, antmicro-footprints:1206-res, symbol antmicroResistorsmisc:R_0R_1206
- added TP? (x5): TP_SMD1MM, lpddr4-test-board-footprints:Testpoint_smd_1mm, symbol lpddr4-test-board:TP_SMD1MM
Connections:
- wire segments 151 -> 157
Other:
- note added: "VDD0V6 0.6V 1.5A"
- note removed: "VDD1V1 0.6V 1.5A"
- moved on the sheet: C?
Changed lines of the file:
@@
 AVCC3V3
-$Comp
-L lpddr4-test-board:R_0R005_1206 R125
-U 1 1 60599ADE
-P 14375 3500
-F 0 "R125" V 14330 3570 60  0000 L CNN
-F 1 "R_0R005_1206" H 14375 3350 60  0001 C CNN
-F 2 "lpddr4-test-board-footprints:1206-res" H 14575 3700 60  0001 L CNN
-F 3 "" H 14375 3500 50  0001 C CNN
-F 4 "WELWYN" H 14575 3900 60  0001 L CNN "Manufacturer"
-F 5 "LRF1206-R005JW" H 14575 3800 60  0001 L CNN "MPN"
-F 6 "0R005" V 14428 3570 50  0000 L CNN "Val"
-	1    14375 3500
-	0    1    1    0
-$EndComp
 $Comp
 L lpddr4-test-board:DC_SOCKET J3
@@
 Wire Wire Line
 	4350 3250 4400 3250
-Text GLabel 6750 2350 2    50   Input ~ 0
+Text GLabel 7175 2350 2    50   Input ~ 0
 VDD1V8
 Wire Wire Line
@@
 Wire Wire Line
 	6225 2800 6225 2650
-Text GLabel 6750 2800 2    50   Input ~ 0
+Text GLabel 7175 2800 2    50   Input ~ 0
 VDD1V1
 Text GLabel 8250 2300 1    50   Input ~ 0
@@
 Wire Wire Line
 	6625 2800 6750 2800
-Text GLabel 6750 3100 2    50   Input ~ 0
+Text GLabel 7175 3100 2    50   Input ~ 0
 VDD0V6
 Wire Wire Line
@@
 Text Notes 2400 2225 0    50   ~ 0
 VCC5V0 4.5V to 5.5V
-Text Notes 6750 2275 0    50   ~ 0
+Text Notes 7025 2275 0    50   ~ 0
 VDD1V8 1.8V 1A
-Text Notes 6775 2725 0    50   ~ 0
+Text Notes 7050 2725 0    50   ~ 0
 VDD1V1 1.1V 8A
-Text Notes 6775 3025 0    50   ~ 0
-VDD1V1 0.6V 1.5A
+Text Notes 7050 3025 0    50   ~ 0
+VDD0V6 0.6V 1.5A
 $Comp
 L lpddr4-test-board:TPS62823DLCT U?
@@
 Wire Wire Line
 	14375 3650 14375 3900
-Text GLabel 11650 6375 1    50   Input ~ 0
+Text GLabel 11650 6250 1    50   Input ~ 0
 VCC5V0
 Wire Wire Line
-	11650 6375 11650 6550
+	11650 6250 11650 6550
 Wire Wire Line
 	11650 6550 11975 6550
@@
 	11650 6700 11650 6550
 Connection ~ 11650 6550
-Text GLabel 11225 6375 1    50   Input ~ 0
+Text GLabel 11225 6250 1    50   Input ~ 0
 VCC5V0
 $Comp
 L lpddr4-test-board:C_2u2_0402 C?
 U 1 1 601A51FF
-P 11225 6525
-F 0 "C?" H 11340 6570 60  0000 L CNN
-F 1 "C_2u2_0402" H 11225 6375 60  0001 C CNN
-F 2 "lpddr4-test-board-footprints:0402-cap" H 11425 6725 60  0001 L CNN
-F 3 "" H 11225 6525 50  0001 C CNN
-F 4 "TDK" H 11425 6925 60  0001 L CNN "Manufacturer"
-F 5 "C1005X5R1A225K050BC" H 11425 6825 60  0001 L CNN "MPN"
-F 6 "2u2" H 11340 6472 50  0000 L CNN "Val"
-	1    11225 6525
+P 11225 6475
+F 0 "C?" H 11340 6520 60  0000 L CNN
+F 1 "C_2u2_0402" H 11225 6325 60  0001 C CNN
+F 2 "lpddr4-test-board-footprints:0402-cap" H 11425 6675 60  0001 L CNN
+F 3 "" H 11225 6475 50  0001 C CNN
+F 4 "TDK" H 11425 6875 60  0001 L CNN "Manufacturer"
+F 5 "C1005X5R1A225K050BC" H 11425 6775 60  0001 L CNN "MPN"
+F 6 "2u2" H 11340 6422 50  0000 L CNN "Val"
+	1    11225 6475
 	1    0    0    -1
 $EndComp
@@
 L lpddr4-test-board:GND #PWR?
 U 1 1 601F9B65
-P 14275 6675
-F 0 "#PWR?" H 14275 6425 50  0001 C CNN
-F 1 "GND" H 14280 6502 50  0000 C CNN
-F 2 "" H 14275 6675 50  0001 C CNN
-F 3 "" H 14275 6675 50  0001 C CNN
-	1    14275 6675
+P 14250 6675
+F 0 "#PWR?" H 14250 6425 50  0001 C CNN
+F 1 "GND" H 14255 6502 50  0000 C CNN
+F 2 "" H 14250 6675 50  0001 C CNN
+F 3 "" H 14250 6675 50  0001 C CNN
+	1    14250 6675
 	1    0    0    -1
 $EndComp
@@
 L lpddr4-test-board:C_10u_0402 C?
 U 1 1 601F8FE9
-P 14275 6525
-F 0 "C?" H 14390 6570 60  0000 L CNN
-F 1 "C_10u_0402" H 14275 6375 60  0001 C CNN
-F 2 "lpddr4-test-board-footprints:0402-cap" H 14475 6725 60  0001 L CNN
-F 3 "" H 14275 6525 50  0001 C CNN
-F 4 "MURATA" H 14475 6925 60  0001 L CNN "Manufacturer"
-F 5 "GRM155R60J106ME44D" H 14475 6825 60  0001 L CNN "MPN"
-F 6 "10u" H 14390 6472 50  0000 L CNN "Val"
-	1    14275 6525
-	1    0    0    -1
-$EndComp
-Text GLabel 14275 6375 1    50   Input ~ 0
+P 14250 6475
+F 0 "C?" H 14365 6520 60  0000 L CNN
+F 1 "C_10u_0402" H 14250 6325 60  0001 C CNN
+F 2 "lpddr4-test-board-footprints:0402-cap" H 14450 6675 60  0001 L CNN
+F 3 "" H 14250 6475 50  0001 C CNN
+F 4 "MURATA" H 14450 6875 60  0001 L CNN "Manufacturer"
+F 5 "GRM155R60J106ME44D" H 14450 6775 60  0001 L CNN "MPN"
+F 6 "10u" H 14365 6422 50  0000 L CNN "Val"
+	1    14250 6475
+	1    0    0    -1
+$EndComp
+Text GLabel 14250 6250 1    50   Input ~ 0
 VCC3V3
 $Comp
@@
 	1    0    0    -1
 $EndComp
-Text GLabel 13775 6375 1    50   Input ~ 0
+Text GLabel 13775 6250 1    50   Input ~ 0
 VCC3V3
-Wire Wire Line
-	13775 6550 13775 6375
 Wire Wire Line
 	13300 6550 13400 6550
@@
 Connection ~ 6225 2800
 Connection ~ 6625 2800
+$Comp
+L antmicroResistorsmisc:R_0R_1206 R?
+U 1 1 6020F9C4
+P 14375 3500
+F 0 "R?" V 14330 3570 60  0000 L CNN
+F 1 "R_0R_1206" H 14375 3350 60  0001 C CNN
+F 2 "antmicro-footprints:1206-res" H 14575 3700 60  0001 L CNN
+F 3 "" H 14375 3500 50  0001 C CNN
+F 4 "MULTICOMP" H 14575 3900 60  0001 L CNN "Manufacturer"
+F 5 "MCMR12X000_PTL" H 14575 3800 60  0001 L CNN "MPN"
+F 6 "0R" V 14428 3570 50  0000 L CNN "Val"
+	1    14375 3500
+	0    1    1    0
+$EndComp
+Text GLabel 14825 3200 1    50   Input ~ 0
+VCC5V0
+$Comp
+L lpddr4-test-board:TP_SMD1MM TP?
+U 1 1 60212554
+P 14825 3300
+F 0 "TP?" V 14730 3347 50  0000 C CNN
+F 1 "TP_SMD1MM" H 14825 3200 50  0001 C CNN
+F 2 "lpddr4-test-board-footprints:Testpoint_smd_1mm" H 15025 3500 60  0001 L CNN
+F 3 "" H 15025 3600 60  0001 L CNN
+	1    14825 3300
+	1    0    0    -1
+$EndComp
+$Comp
+L antmicroResistorsmisc:R_0R_1206 R?
+U 1 1 6021B240
+P 13775 6400
+F 0 "R?" V 13730 6470 60  0000 L CNN
+F 1 "R_0R_1206" H 13775 6250 60  0001 C CNN
+F 2 "antmicro-footprints:1206-res" H 13975 6600 60  0001 L CNN
+F 3 "" H 13775 6400 50  0001 C CNN
+F 4 "MULTICOMP" H 13975 6800 60  0001 L CNN "Manufacturer"
+F 5 "MCMR12X000_PTL" H 13975 6700 60  0001 L CNN "MPN"
+F 6 "0R" V 13828 6470 50  0000 L CNN "Val"
+	1    13775 6400
+	0    1    1    0
+$EndComp
+Wire Wire Line
+	11225 6250 11225 6325
+Wire Wire Line
+	11225 6625 11225 6675
+Wire Wire Line
+	14250 6250 14250 6325
+Wire Wire Line
+	14250 6625 14250 6675
+Text GLabel 14650 6250 1    50   Input ~ 0
+VCC3V3
+$Comp
+L lpddr4-test-board:TP_SMD1MM TP?
+U 1 1 6026C4D0
+P 14650 6350
+F 0 "TP?" V 14555 6397 50  0000 C CNN
+F 1 "TP_SMD1MM" H 14650 6250 50  0001 C CNN
+F 2 "lpddr4-test-board-footprints:Testpoint_smd_1mm" H 14850 6550 60  0001 L CNN
+F 3 "" H 14850 6650 60  0001 L CNN
+	1    14650 6350
+	1    0    0    -1
+$EndComp
+$Comp
+L antmicroResistorsmisc:R_0R_1206 R?
+U 1 1 60283299
+P 6900 2350
+F 0 "R?" H 6900 2137 60  0000 C CNN
+F 1 "R_0R_1206" H 6900 2200 60  0001 C CNN
+F 2 "antmicro-footprints:1206-res" H 7100 2550 60  0001 L CNN
+F 3 "" H 6900 2350 50  0001 C CNN
+F 4 "MULTICOMP" H 7100 2750 60  0001 L CNN "Manufacturer"
+F 5 "MCMR12X000_PTL" H 7100 2650 60  0001 L CNN "MPN"
+F 6 "0R" H 6900 2235 50  0000 C CNN "Val"
+	1    6900 2350
+	-1   0    0    1
+$EndComp
+$Comp
+L antmicroResistorsmisc:R_0R_1206 R?
+U 1 1 60285989
+P 6900 2800
+F 0 "R?" H 6900 2587 60  0000 C CNN
+F 1 "R_0R_1206" H 6900 2650 60  0001 C CNN
+F 2 "antmicro-footprints:1206-res" H 7100 3000 60  0001 L CNN
+F 3 "" H 6900 2800 50  0001 C CNN
+F 4 "MULTICOMP" H 7100 3200 60  0001 L CNN "Manufacturer"
+F 5 "MCMR12X000_PTL" H 7100 3100 60  0001 L CNN "MPN"
+F 6 "0R" H 6900 2685 50  0000 C CNN "Val"
+	1    6900 2800
+	-1   0    0    1
+$EndComp
+$Comp
+L antmicroResistorsmisc:R_0R_1206 R?
+U 1 1 60285DF8
+P 6900 3100
+F 0 "R?" H 6900 2887 60  0000 C CNN
+F 1 "R_0R_1206" H 6900 2950 60  0001 C CNN
+F 2 "antmicro-footprints:1206-res" H 7100 3300 60  0001 L CNN
+F 3 "" H 6900 3100 50  0001 C CNN
+F 4 "MULTICOMP" H 7100 3500 60  0001 L CNN "Manufacturer"
+F 5 "MCMR12X000_PTL" H 7100 3400 60  0001 L CNN "MPN"
+F 6 "0R" H 6900 2985 50  0000 C CNN "Val"
+	1    6900 3100
+	-1   0    0    1
+$EndComp
+Wire Wire Line
+	7175 2350 7050 2350
+Wire Wire Line
+	7175 2800 7050 2800
+Wire Wire Line
+	7175 3100 7050 3100
+Text GLabel 6800 3650 1    50   Input ~ 0
+VDD1V8
+Text GLabel 7025 3650 1    50   Input ~ 0
+VDD1V1
+Text GLabel 7250 3650 1    50   Input ~ 0
+VDD0V6
+$Comp
+L lpddr4-test-board:TP_SMD1MM TP?
+U 1 1 602C0646
+P 6800 3750
+F 0 "TP?" V 6705 3797 50  0000 C CNN
+F 1 "TP_SMD1MM" H 6800 3650 50  0001 C CNN
+F 2 "lpddr4-test-board-footprints:Testpoint_smd_1mm" H 7000 3950 60  0001 L CNN
+F 3 "" H 7000 4050 60  0001 L CNN
+	1    6800 3750
+	1    0    0    -1
+$EndComp
+$Comp
+L lpddr4-test-board:TP_SMD1MM TP?
+U 1 1 602C252D
+P 7025 3750
+F 0 "TP?" V 6930 3797 50  0000 C CNN
+F 1 "TP_SMD1MM" H 7025 3650 50  0001 C CNN
+F 2 "lpddr4-test-board-footprints:Testpoint_smd_1mm" H 7225 3950 60  0001 L CNN
+F 3 "" H 7225 4050 60  0001 L CNN
+	1    7025 3750
+	1    0    0    -1
+$EndComp
+$Comp
+L lpddr4-test-board:TP_SMD1MM TP?
+U 1 1 602C27EC
+P 7250 3750
+F 0 "TP?" V 7155 3797 50  0000 C CNN
+F 1 "TP_SMD1MM" H 7250 3650 50  0001 C CNN
+F 2 "lpddr4-test-board-footprints:Testpoint_smd_1mm" H 7450 3950 60  0001 L CNN
+F 3 "" H 7450 4050 60  0001 L CNN
+	1    7250 3750
+	1    0    0    -1
+$EndComp
 $EndSCHEMATC

Commit message: Library cleanup, add RGMII layout
Parts:
- R43, R44, R45, R46, R49: renamed from R?; footprint antmicro-footprints:1206-res -> lpddr4-test-board-footprints:1206-res; symbol antmicroResistorsmisc:R_0R_1206 -> lpddr4-test-board:R_0R_1206
- gave numbers to parts that had none: 37
