File: hyperram.sch (KiCad schematic (older format))
At the start: 7 parts, among them U11 S27KL0641DABHI023

Commit message: Update local libraries
Parts:
- U11: footprint antmicro-footprints:FBGA-24 -> lpddr4-test-board-footprints:FBGA-24
Changed lines of the file:
@@
 F 0 "U11" H 3800 5315 50  0000 C CNN
 F 1 "S27KL0641DABHI023" H 3800 5224 50  0000 C CNN
-F 2 "antmicro-footprints:FBGA-24" H 3350 3250 50  0001 L BNN
+F 2 "lpddr4-test-board-footprints:FBGA-24" H 3350 3250 50  0001 L BNN
 F 3 "" H 3800 4350 50  0001 L BNN
 F 4 "CYPRESS SEMICONDUCTOR" H 3850 3100 50  0001 C CNN "Manufacturer"
