File: config-spi.sch (KiCad schematic (older format))
At the start: 38 parts, among them J1 0878311420, Q7 BSS138APW, Q8 BSS138APW, U1 XC7K70T-FBG484, U3 S25FL128SAGNFI000

Commit message: Update MPNs, add BOM
Parts:
- U1: MPN (none) -> XC7K70T-1FBG484C; Manufacturer (none) -> Xilinx
- U3: MPN (none) -> S25FL128SAGNFI000; Manufacturer (none) -> Cypress Semiconductor
Changed lines of the file:
@@
 F 2 "lpddr4-test-board-footprints:BGA484C100P22X22_2300X2300X244N" H 13175 5300 50  0001 C CNN
 F 3 "" H 13175 5300 50  0000 C CNN
+F 4 "XC7K70T-1FBG484C" H 13175 5300 50  0001 C CNN "MPN"
+F 5 "Xilinx" H 13175 5300 50  0001 C CNN "Manufacturer"
 	6    13175 5300
 	-1   0    0    -1
@@
 F 2 "lpddr4-test-board-footprints:S25FL128SAGNFI000" H 5300 4390 60  0001 C CNN
 F 3 "" H 4300 4150 60  0000 C CNN
+F 4 "S25FL128SAGNFI000" H 4300 4150 50  0001 C CNN "MPN"
+F 5 "Cypress Semiconductor" H 4300 4150 50  0001 C CNN "Manufacturer"
 	1    4300 4150
 	-1   0    0    -1
