File: ethernet.kicad_sch (KiCad schematic)
At the start: 57 parts, among them J5 WE-RJ45_7499111121A, U6 KSZ9031RNXCA, Y2 ABM8G-25.000MHZ-18-D2Y-T

Commit message: Introduce standardized components
Parts:
- C100, C103, C104, C105, C98: footprint lpddr4-test-board-footprints:0402-cap -> lpddr4-test-board-footprints:C_0402_1005Metric; Author (none) -> Antmicro; License (none) -> Apache-2.0
- C101, C102, C110, C97, C99: footprint lpddr4-test-board-footprints:0402-cap -> lpddr4-test-board-footprints:C_0402_1005Metric; Author (none) -> Antmicro; License (none) -> Apache-2.0; Manufacturer MURATA -> Murata
- C106: value C_100n_0402 -> C_100n_16V_0402; footprint lpddr4-test-board-footprints:0402-cap -> lpddr4-test-board-footprints:C_0402_1005Metric; symbol lpddr4-test-board:C_100n_0402_16V -> lpddr4-test-board:C_100n_16V_0402; Author (none) -> Antmicro; License (none) -> Apache-2.0; Manufacturer MULTICOMP -> Multicomp
- C107, C109, C111, C112, C113, C114, C116, C117, C119, C120: footprint lpddr4-test-board-footprints:0402-cap -> lpddr4-test-board-footprints:C_0402_1005Metric; Author (none) -> Antmicro; Dielectric (none) -> X7R; License (none) -> Apache-2.0; MPN 04025G103ZAT2A -> GRM155R71H103KA88D; Manufacturer AVX -> Murata; Voltage (none) -> 50V
- C108: value C_10n_0402 -> C_470n_0402; footprint lpddr4-test-board-footprints:0402-cap -> lpddr4-test-board-footprints:C_0402_1005Metric; Author (none) -> Antmicro; License (none) -> Apache-2.0
- C115, C118: value C_10n_0402 -> C_4u7_0402; footprint lpddr4-test-board-footprints:0402-cap -> lpddr4-test-board-footprints:C_0402_1005Metric; Author (none) -> Antmicro; License (none) -> Apache-2.0; Manufacturer MURATA -> Murata
- C121, C122: footprint lpddr4-test-board-footprints:0402-cap -> lpddr4-test-board-footprints:C_0402_1005Metric; Author (none) -> Antmicro; License (none) -> Apache-2.0; Manufacturer YAGEO -> Yaego
- FB4, FB5, FB6, FB7: value BLM18PG121SN1D -> FB_120Z_2A_0603; footprint lpddr4-test-board-footprints:0603-res -> lpddr4-test-board-footprints:FB_0603_1608Metric; symbol lpddr4-test-board:BLM18PG121SN1D -> lpddr4-test-board:FB_120Z_2A_0603; Author (none) -> Antmicro; License (none) -> Apache-2.0; Manufacturer Murata Electronics North America -> Murata
- J5: value WE-RJ45_7499111121A -> Bus_RJ45_7499111121A; footprint lpddr4-test-board-footprints:7499111121A -> lpddr4-test-board-footprints:RJ45_7499111121A_Horizontal; symbol lpddr4-test-board:WE-RJ45_7499111121A -> lpddr4-test-board:Bus_RJ45_7499111121A; Author (none) -> Antmicro; License (none) -> Apache-2.0; Manufacturer WURTH ELEKTRONIK -> Würth Elektronik
- R70, R71: footprint lpddr4-test-board-footprints:0402-res -> lpddr4-test-board-footprints:R_0402_1005Metric; Author (none) -> Antmicro; License (none) -> Apache-2.0; MPN ERJ2GEJ221X -> CR0402-FX-2200GLF; Manufacturer Panasonic -> Bourns; Tolerance (none) -> 1%
- R72: footprint lpddr4-test-board-footprints:0402-res -> lpddr4-test-board-footprints:R_0402_1005Metric; Author (none) -> Antmicro; License (none) -> Apache-2.0; MPN MCWR04X1212FTL -> CR0402-FX-1212GLF; Manufacturer MULTICOMP -> Bourns; Tolerance (none) -> 1%
- R73: footprint lpddr4-test-board-footprints:0402-res -> lpddr4-test-board-footprints:R_0402_1005Metric; Author (none) -> Antmicro; License (none) -> Apache-2.0; MPN MCMR04X185_JTL -> CR0402-FX-1804GLF; Manufacturer MULTICOMP -> Bourns; Tolerance (none) -> 1%
- R74, R75, R76, R77, R78, R79, R80, R81, R82, R84: footprint lpddr4-test-board-footprints:0402-res -> lpddr4-test-board-footprints:R_0402_1005Metric; Author (none) -> Antmicro; License (none) -> Apache-2.0; MPN MCWR04X1022FTL -> CR0402-FX-1022GLF; Manufacturer MULTICOMP PRO -> Bourns; Tolerance (none) -> 1%
- R83: footprint lpddr4-test-board-footprints:0402-res -> lpddr4-test-board-footprints:R_0402_1005Metric; Author (none) -> Antmicro; License (none) -> Apache-2.0; Manufacturer BOURNS -> Bourns; Tolerance (none) -> 1%
- R85, R86, R87, R88, R89, R90, R91, R92, R93: footprint lpddr4-test-board-footprints:0402-res -> lpddr4-test-board-footprints:R_0402_1005Metric; Author (none) -> Antmicro; License (none) -> Apache-2.0; MPN RC0402FR-072K2L -> CR0402-FX-2201GLF; Manufacturer YAGEO -> Bourns; Tolerance (none) -> 1%
- U6: footprint lpddr4-test-board-footprints:QFN-48-Microchip-QFN77-48LD-PL-2 -> lpddr4-test-board-footprints:QFN-48-1EP_7x7x0.9mm_P0.5mm_EP3.5x3.5mm; Author (none) -> Antmicro; License (none) -> Apache-2.0
- Y2: value ABM8G-25.000MHZ-18-D2Y-T -> Oscillator_SMD_25MHz_KX-7; footprint lpddr4-test-board-footprints:KX-7 -> lpddr4-test-board-footprints:Oscillator_SMD_Geyer_KX-7-4Pin_3.2x2.5mm; symbol lpddr4-test-board:ABM8G-25.000MHZ-18-D2Y-T -> lpddr4-test-board:Oscillator_SMD_25MHz_KX-7; Author (none) -> Antmicro; License (none) -> Apache-2.0; Val (none) -> 25MHz
Connections:
- net 1V2_SYS: now also FB5.1, FB6.1; no longer FB5.2, FB6.2
- net AVDDL: now also FB6.2; no longer FB6.1
- net AVDDL_PLL: now also FB5.2; no longer FB5.1
- net ETH_XO: now reaches C121.1, R73.1, U6.45 (XO), Y2.1
- net ETH_XI: now reaches C122.1, R73.2, U6.46 (XI), Y2.3
- net at U6.13 (NC): now also U6.47 (NC)
- new net: FB7.1, J5.SH
- no-connect marks 1 -> 2
Other:
- moved on the sheet: C100, C101, C102, C103, C104, C105, C106, C107, C108, C109, C110, C111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

Commit message: [#55158] components update
Parts:
- R74, R75, R78, R79, R87, R88, R91, R92, R93: now not fitted; now left out of the parts list
- R90: DNP DNP -> (none)
- U6: Manufacturer Microchip -> Microchip Technology
- Y2: symbol lpddr4-test-board:Oscillator_SMD_25MHz_KX-7 -> lpddr4-test-board:Resonator_25MHz_ABM8G; MPN ABM8G-25.000MHZ-18-D2Y-T -> ABM8G-25.000MHZ-18-D2Y-T3; Val 25MHz -> 25 MHz
Connections:
- net at U6.13 (NC): no longer U6.47 (NC)
