File: fpga-banks.kicad_sch (KiCad schematic)
At the start: 9 parts, among them U2 ASFL1-100.000MHZ-L-T, U3 XC7K70T-FBG484

Commit message: Loclib
Parts:
- U2: footprint antmicro-footprints:Oscillator_SMD_Abracon_ASFL1-4Pin_5.0x3.2mm -> lpddr4-test-board-footprints:Oscillator_SMD_Abracon_ASFL1-4Pin_5.0x3.2mm; symbol antmicroOscillators:ASFL1-100.000MHZ-L-T -> lpddr4-test-board:ASFL1-100.000MHZ-L-T
Changed lines of the file:
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@@
     )
     (property "Value" "GND" (id 1) (at 344.678 236.8042 0))
-    (property "Footprint" "" (id 2) (at 344.805 232.41 0)
+    (property "Footprint" "lpddr4-test-board-footprints:" (id 2) (at 344.805 232.41 0)
       (effects (font (size 1.27 1.27)) hide)
     )
@@
     )
     (property "Value" "GND" (id 1) (at 356.743 236.8042 0))
-    (property "Footprint" "" (id 2) (at 356.87 232.41 0)
+    (property "Footprint" "lpddr4-test-board-footprints:" (id 2) (at 356.87 232.41 0)
       (effects (font (size 1.27 1.27)) hide)
     )
@@
     )
     (property "Value" "GND" (id 1) (at 366.903 236.8042 0))
-    (property "Footprint" "" (id 2) (at 367.03 232.41 0)
+    (property "Footprint" "lpddr4-test-board-footprints:" (id 2) (at 367.03 232.41 0)
       (effects (font (size 1.27 1.27)) hide)
     )
@@
     )
     (property "Value" "GND" (id 1) (at 330.073 232.3592 0))
-    (property "Footprint" "" (id 2) (at 330.2 227.965 0)
+    (property "Footprint" "lpddr4-test-board-footprints:" (id 2) (at 330.2 227.965 0)
       (effects (font (size 1.27 1.27)) hide)
     )
@@
     )
     (property "Value" "GND" (id 1) (at 86.868 263.4742 0))
-    (property "Footprint" "" (id 2) (at 86.995 259.08 0)
+    (property "Footprint" "lpddr4-test-board-footprints:" (id 2) (at 86.995 259.08 0)
       (effects (font (size 1.27 1.27)) hide)
     )
@@
     )
     (property "Value" "GND" (id 1) (at 33.528 264.1092 0))
-    (property "Footprint" "" (id 2) (at 33.655 259.715 0)
+    (property "Footprint" "lpddr4-test-board-footprints:" (id 2) (at 33.655 259.715 0)
       (effects (font (size 1.27 1.27)) hide)
     )
@@
     (pin "1")
   )
-  (symbol (lib_id "antmicroOscillators:ASFL1-100.000MHZ-L-T") (at 36.195 255.905 0) (unit 1)
+  (symbol (lib_id "lpddr4-test-board:ASFL1-100.000MHZ-L-T") (at 36.195 255.905 0) (unit 1)
     (in_bom yes) (on_board yes) (fields_autoplaced)
     (property "Reference" "U2" (id 0) (at 52.07 249.2809 0)
@@
       (effects (font (size 1.524 1.524)))
     )
-    (property "Footprint" "antmicro-footprints:Oscillator_SMD_Abracon_ASFL1-4Pin_5.0x3.2mm" (id 2) (at 52.07 262.89 0)
-      (effects (font (size 1.524 1.524)) hide)
-    )
+    (property "Footprint" "lpddr4-test-board-footprints:Oscillator_SMD_Abracon_ASFL1-4Pin_5.0x3.2mm" (id 2) (at 52.07 262.89 0)
+      (effects (font (size 1.524 1.524)) hide)
+    )

Commit message: Introduce standardized components
Parts:
- removed unit 1 of U3
- removed unit 2 of U3
- added unit 4 of U3
- added unit 6 of U3
- added unit 9 of U3
- added unit 5 of U3
- added unit 7 of U3
- added unit 8 of U3
- C5, C6, C7: value C_100n_0402_6V3 -> C_100n_6V3_0402; footprint lpddr4-test-board-footprints:0402-cap -> lpddr4-test-board-footprints:C_0402_1005Metric; symbol lpddr4-test-board:C_100n_0402_6V3 -> lpddr4-test-board:C_100n_6V3_0402; Author (none) -> Antmicro; License (none) -> Apache-2.0
- R3, R4: footprint lpddr4-test-board-footprints:0603-res -> lpddr4-test-board-footprints:R_0603_1608Metric; Author (none) -> Antmicro; License (none) -> Apache-2.0; MPN CRCW0603120RFKEA -> CR0603-FX-1200ELF; Manufacturer VISHAY -> Bourns; Tolerance (none) -> 1%
- R5, R6: footprint lpddr4-test-board-footprints:0603-res -> lpddr4-test-board-footprints:R_0603_1608Metric; Author (none) -> Antmicro; License (none) -> Apache-2.0; MPN CR0603-JW-102ELF -> CR0603-FX-1001ELF; Manufacturer BOURNS -> Bourns; Tolerance (none) -> 1%
- U2, U3: Author (none) -> Antmicro; License (none) -> Apache-2.0
Connections:
- net 3V3_SYS: now also C5.2; no longer C5.1
- net AUX_JTAG_RST: now also U3.AB17 (IO_L17N_T2_13)
- net AUX_JTAG_TCK: now also U3.W22 (IO_L4N_T0_13)
- net AUX_JTAG_TDI: now also U3.W20 (IO_L11N_T1_SRCC_13)
- net AUX_JTAG_TDO: now also U3.W21 (IO_L4P_T0_13)
- net AUX_JTAG_TMS: now also U3.Y21 (IO_L7P_T1_13)
- net CA2_A: now also U3.AA4 (IO_L24P_T3_34); no longer U3.AA4 (IO_L24P_T3_34)
- net CA3_A: now also U3.AA3 (IO_L23P_T3_34); no longer U3.AA3 (IO_L23P_T3_34)
- net CA4_A: now also U3.AB3 (IO_L24N_T3_34); no longer U3.AB3 (IO_L24N_T3_34)
- net CA5_A: now also U3.AB2 (IO_L23N_T3_34); no longer U3.AB2 (IO_L23N_T3_34)
- net CA_0A: now also U3.L3 (IO_L1P_T0_34); no longer U3.L3 (IO_L1P_T0_34)
- net CA_1A: now also U3.L5 (IO_L6P_T0_34); no longer U3.L5 (IO_L6P_T0_34)
- net CKE0_A: now also U3.N4 (IO_L9N_T1_DQS_34); no longer U3.N4 (IO_L9N_T1_DQS_34)
- net CK_A_N: now also U3.Y2 (IO_L21N_T3_DQS_34); no longer U3.Y2 (IO_L21N_T3_DQS_34)
- net CK_A_P: now also U3.Y3 (IO_L21P_T3_DQS_34); no longer U3.Y3 (IO_L21P_T3_DQS_34)
- net CS0_A: now also U3.N3 (IO_L5P_T0_34); no longer U3.N3 (IO_L5P_T0_34)
- net DMI_0A: now also U3.M3 (IO_L1N_T0_34); no longer U3.M3 (IO_L1N_T0_34)
- net DMI_1A: now also U3.W1 (IO_L20P_T3_34); no longer U3.W1 (IO_L20P_T3_34)
- net DQ00_A: now also U3.L1 (IO_L2N_T0_34); no longer U3.L1 (IO_L2N_T0_34)
- net DQ01_A: now also U3.K2 (IO_L4N_T0_34); no longer U3.K2 (IO_L4N_T0_34)
- net DQ02_A: now also U3.K1 (IO_L2P_T0_34); no longer U3.K1 (IO_L2P_T0_34)
- net DQ03_A: now also U3.K3 (IO_L4P_T0_34); no longer U3.K3 (IO_L4P_T0_34)
- net DQ04_A: now also U3.R1 (IO_L8N_T1_34); no longer U3.R1 (IO_L8N_T1_34)
- net DQ05_A: now also U3.P2 (IO_L7P_T1_34); no longer U3.P2 (IO_L7P_T1_34)
- net DQ06_A: now also U3.P1 (IO_L8P_T1_34); no longer U3.P1 (IO_L8P_T1_34)
- net DQ07_A: now also U3.N2 (IO_L5N_T0_34); no longer U3.N2 (IO_L5N_T0_34)
- net DQ08_A: now also U3.W2 (IO_L17N_T2_34); no longer U3.W2 (IO_L17N_T2_34)
- net DQ09_A: now also U3.Y1 (IO_L20N_T3_34); no longer U3.Y1 (IO_L20N_T3_34)
- net DQ10_A: now also U3.AA1 (IO_L22P_T3_34); no longer U3.AA1 (IO_L22P_T3_34)
- net DQ11_A: now also U3.AB1 (IO_L22N_T3_34); no longer U3.AB1 (IO_L22N_T3_34)
- net DQ12_A: now also U3.R2 (IO_L7N_T1_34); no longer U3.R2 (IO_L7N_T1_34)
- net DQ13_A: now also U3.T1 (IO_L10P_T1_34); no longer U3.T1 (IO_L10P_T1_34)
- net DQ14_A: now also U3.T3 (IO_L12N_T1_MRCC_34); no longer U3.T3 (IO_L12N_T1_MRCC_34)
- net DQ15_A: now also U3.U1 (IO_L10N_T1_34); no longer U3.U1 (IO_L10N_T1_34)
- net DQ_S0_N: now also U3.M1 (IO_L3N_T0_DQS_34); no longer U3.M1 (IO_L3N_T0_DQS_34)
- net DQ_S0_P: now also U3.M2 (IO_L3P_T0_DQS_34); no longer U3.M2 (IO_L3P_T0_DQS_34)
- net DQ_S1_N: now also U3.V2 (IO_L15N_T2_DQS_34); no longer U3.V2 (IO_L15N_T2_DQS_34)
- net DQ_S1_P: now also U3.U2 (IO_L15P_T2_DQS_34); no longer U3.U2 (IO_L15P_T2_DQS_34)
- net EMCCLK: now also U3.J19 (IO_L3N_T0_DQS_EMCCLK_14)
- net ETH_INT_N: now also U3.C15 (IO_L7N_T1_AD10N_15)
- net ETH_MDC: now also U3.B17 (IO_L10P_T1_AD4P_15)
- net ETH_MDIO: now also U3.C14 (IO_L7P_T1_AD10P_15)
- net ETH_REF_CLK: now also U3.C12 (IO_L2P_T0_AD8P_15)
- net ETH_RSTN: now also U3.E16 (IO_L14P_T2_SRCC_15)
- net ETH_RXD0: now also U3.B16 (IO_L8P_T1_AD3P_15)
- net ETH_RXD1: now also U3.A15 (IO_L9N_T1_DQS_AD11N_15)
- net ETH_RXD2: now also U3.B15 (IO_L9P_T1_DQS_AD11P_15)
- net ETH_RXD3: now also U3.A14 (IO_L4N_T0_AD9N_15)
- net ETH_RX_CLK: now also U3.C17 (IO_L12P_T1_MRCC_AD5P_15)
- net ETH_RX_DV: now also U3.A16 (IO_L8N_T1_AD3N_15)
- net ETH_TXD0: now also U3.B21 (IO_L24N_T3_RS0_15)
- net ETH_TXD1: now also U3.B20 (IO_L24P_T3_RS1_15)
- net ETH_TXD2: now also U3.A19 (IO_L20N_T3_A19_15)
- net ETH_TXD3: now also U3.A18 (IO_L10N_T1_AD4N_15)
- net ETH_TX_CLK: now also U3.E17 (IO_L13P_T2_MRCC_15)
- net ETH_TX_EN: now also U3.A13 (IO_L4P_T0_AD9P_15)
- net FCS_B: now also U3.L16 (IO_L6P_T0_FCS_B_14)
- net FPGA_AA21_BALL: now also U3.AA21 (IO_L9P_T1_DQS_13)
- net FPGA_AB21_BALL: now also U3.AB21 (IO_L8N_T1_13)
- net FPGA_AB22_BALL: now also U3.AB22 (IO_L9N_T1_DQS_13)
- net GCLK100: now also U3.L19 (IO_L12P_T1_MRCC_14)
- net GND: now also C5.1, C6.1, C7.1; no longer C5.2, C6.2, C7.2
- net HR_CKN: now also U3.AB16 (IO_L16N_T2_13)
- net HR_CKP: now also U3.AB15 (IO_L16P_T2_13)
- net HR_CS: now also U3.AA16 (IO_L17P_T2_13)
- net HR_DQ0: now also U3.W15 (IO_L23N_T3_13)
- net HR_DQ1: now also U3.AA15 (IO_L18N_T2_13)
- net HR_DQ2: now also U3.AA14 (IO_L18P_T2_13)
- net HR_DQ3: now also U3.W14 (IO_L22P_T3_13)
- net HR_DQ4: now also U3.Y14 (IO_L22N_T3_13)
- net HR_DQ5: now also U3.V15 (IO_L23P_T3_13)
- net HR_DQ6: now also U3.Y16 (IO_L21N_T3_DQS_13)
- net HR_DQ7: now also U3.W17 (IO_L14P_T2_SRCC_13)
- net HR_RST: now also U3.V17 (IO_L19N_T3_VREF_13)
- net HR_RW: now also U3.Y17 (IO_L14N_T2_SRCC_13)
- net IO_AA11: now also U3.AA11 (IO_L20P_T3_33); no longer U3.AA11 (IO_L20P_T3_33)
- net IO_AB10: now also U3.AB10 (IO_L4N_T0_33); no longer U3.AB10 (IO_L4N_T0_33)
- net IO_AB11: now also U3.AB11 (IO_L20N_T3_33); no longer U3.AB11 (IO_L20N_T3_33)
- net IO_M5: now also U3.M5 (IO_L9P_T1_DQS_34); no longer U3.M5 (IO_L9P_T1_DQS_34)
- net IO_N5: now also U3.N5 (IO_L18P_T2_34); no longer U3.N5 (IO_L18P_T2_34)
- net IO_P4: now also U3.P4 (IO_L11P_T1_SRCC_34); no longer U3.P4 (IO_L11P_T1_SRCC_34)
- net IO_R4: now also U3.R4 (IO_L11N_T1_SRCC_34); no longer U3.R4 (IO_L11N_T1_SRCC_34)
- net IO_T4: now also U3.T4 (IO_L13P_T2_MRCC_34); no longer U3.T4 (IO_L13P_T2_MRCC_34)
- net IO_U12: now also U3.U12 (IO_L17P_T2_33); no longer U3.U12 (IO_L17P_T2_33)
- net IO_U3: now also U3.U3 (IO_L13N_T2_MRCC_34); no longer U3.U3 (IO_L13N_T2_MRCC_34)
- net IO_U5: now also U3.U5 (IO_L16N_T2_34); no longer U3.U5 (IO_L16N_T2_34)
- net IO_V12: now also U3.V12 (IO_L23N_T3_33); no longer U3.V12 (IO_L23N_T3_33)
- net IO_V3: now also U3.V3 (IO_L17P_T2_34); no longer U3.V3 (IO_L17P_T2_34)
- net IO_V4: now also U3.V4 (IO_L14P_T2_SRCC_34); no longer U3.V4 (IO_L14P_T2_SRCC_34)
- net IO_W11: now also U3.W11 (IO_L6P_T0_33); no longer U3.W11 (IO_L6P_T0_33)
- net IO_W12: now also U3.W12 (IO_L19P_T3_33); no longer U3.W12 (IO_L19P_T3_33)
- net IO_W4: now also U3.W4 (IO_L14N_T2_SRCC_34); no longer U3.W4 (IO_L14N_T2_SRCC_34)
- net IO_Y11: now also U3.Y11 (IO_L6N_T0_VREF_33); no longer U3.Y11 (IO_L6N_T0_VREF_33)
- net IO_Y12: now also U3.Y12 (IO_L19N_T3_VREF_33); no longer U3.Y12 (IO_L19N_T3_VREF_33)
- net PUDC_B: now also U3.K18 (IO_L3P_T0_DQS_PUDC_B_14)
- net QSPI_DQ0: now also U3.H18 (IO_L1P_T0_D00_MOSI_14)
- net QSPI_DQ1: now also U3.H19 (IO_L1N_T0_D01_DIN_14)
- net QSPI_DQ2: now also U3.G18 (IO_L2P_T0_D02_14)
- net QSPI_DQ3: now also U3.F19 (IO_L2N_T0_D03_14)
- net SD_CD: now also U3.B22 (IO_L21N_T3_DQS_A18_15)
- net SD_CLK: now also U3.D22 (IO_L23N_T3_FWE_B_15)
- net SD_CMD: now also U3.C20 (IO_L19N_T3_A21_VREF_15)
- net SD_DAT0: now also U3.D21 (IO_L23P_T3_FOE_B_15)
- net SD_DAT1: now also U3.C22 (IO_L21P_T3_DQS_15)
- net SD_DAT2: now also U3.D19 (IO_L18P_T2_A24_15)
- net SD_DAT3: now also U3.D20 (IO_L18N_T2_A23_15)
- net TMDS_CLK_N: now also U3.R22 (IO_L24N_T3_A00_D16_14)
- net TMDS_CLK_P: now also U3.R21 (IO_L24P_T3_A01_D17_14)
- net TMDS_D0_N: now also U3.P22 (IO_L22N_T3_A04_D20_14)
- net TMDS_D0_P: now also U3.P21 (IO_L22P_T3_A05_D21_14)
- net TMDS_D1_N: now also U3.K22 (IO_L16N_T2_A15_D31_14)
- net TMDS_D1_P: now also U3.K21 (IO_L16P_T2_CSI_B_14)
- net TMDS_D2_N: now also U3.J22 (IO_L10N_T1_D15_14)
- net TMDS_D2_P: now also U3.J21 (IO_L10P_T1_D14_14)
- net UART0_RX: now also U3.AA18 (IO_L15P_T2_DQS_13)
- net UART0_TX: now also U3.AB18 (IO_L15N_T2_DQS_13)
- net UART1_RX: now also U3.AB20 (IO_L10N_T1_13)
- net UART1_TX: now also U3.AA20 (IO_L8P_T1_13)
- net USR_BTN1: now also U3.E8 (IO_24_T3_16)
- net USR_BTN2: now also U3.B8 (IO_L22N_T3_16)
- net USR_BTN3: now also U3.C9 (IO_L19N_T3_VREF_16)
- net USR_BTN4: now also U3.E9 (IO_L15N_T2_DQS_16)
- net USR_LED1: now also U3.F8 (IO_L17N_T2_16)
- net USR_LED2: now also U3.C8 (IO_L22P_T3_16)
- net USR_LED3: now also U3.A8 (IO_L21N_T3_DQS_16)
- net USR_LED4: now also U3.D9 (IO_L19P_T3_16)
- net USR_LED5: now also U3.F9 (IO_L15P_T2_DQS_16)
- net VDDQ: no longer U3.AA7 (VCCO_33), U3.AB4 (VCCO_34), U3.M4 (VCCO_34), U3.N1 (VCCO_34), U3.R5 (VCCO_34), U3.T12 (VCCO_33), U3.T2 (VCCO_34), U3.U9 (VCCO_33), U3.V6 (VCCO_33), U3.W13 (VCCO_33), U3.W3 (VCCO_34), U3.Y10 (VCCO_33)
- net VREF_34: now also C6.2, C7.2, U3.L4 (IO_L6N_T0_VREF_34), U3.Y4 (IO_L19N_T3_VREF_34); no longer C6.1, C7.1, U3.L4 (IO_L6N_T0_VREF_34), U3.Y4 (IO_L19N_T3_VREF_34)
- net VRN: now also U3.K4 (IO_0_VRN_34); no longer U3.K4 (IO_0_VRN_34)
- net VRP: now also U3.V5 (IO_25_VRP_34); no longer U3.V5 (IO_25_VRP_34)
- no-connect marks 29 -> 176
Other:
- note added: "UNUSED"
- note removed: "VCCO (HP banks) max: 2.0V"
- note removed: "VCCO (HR banks) max: 3.6V"
- moved on the sheet: C5, C6, C7, R3, R4, R5, R6, U2

Commit message: [#55158] components update
Parts:
- U2: symbol lpddr4-test-board:ASFL1-100.000MHZ-L-T -> lpddr4-test-board:Oscillator_100MHz_ASFL1; Val (none) -> 100 MHz
- U3: Manufacturer Xilinx -> AMD-Xilinx
