File: interfaces.kicad_sch (KiCad schematic)
At the start: 84 parts, among them IC1 TPD8S009DSMR, J1 WE_629105150521, J2 685119134923, J3 1140084168, Q1 BSS138APW, Q2 BSS138APW, Q3 BSS138APW, Q4 BSS138APW, Q5 BSS138APW, U4 FT4232H-56Q, Y1 ABM8G-12.000MHZ-18-D2Y-T

Commit message: Loclib
Parts:
- U4: footprint antmicro-footprints:QFN-56-1EP_8x8mm_P0.5mm_EP5.5.9x5.9mm -> lpddr4-test-board-footprints:QFN-56-1EP_8x8mm_P0.5mm_EP5.5.9x5.9mm; symbol antmicroInterfaceControllers:FT4232H-56Q -> lpddr4-test-board:FT4232H-56Q
Changed lines of the file:
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@@
     )
     (property "Value" "GND" (id 1) (at 136.652 269.8242 0))
-    (property "Footprint" "" (id 2) (at 136.525 265.43 0)
+    (property "Footprint" "lpddr4-test-board-footprints:" (id 2) (at 136.525 265.43 0)
       (effects (font (size 1.27 1.27)) hide)
     )
@@
     )
     (property "Value" "GND" (id 1) (at 111.252 269.8242 0))
-    (property "Footprint" "" (id 2) (at 111.125 265.43 0)
+    (property "Footprint" "lpddr4-test-board-footprints:" (id 2) (at 111.125 265.43 0)
       (effects (font (size 1.27 1.27)) hide)
     )
@@
     )
     (property "Value" "GND" (id 1) (at 97.917 269.8242 0))
-    (property "Footprint" "" (id 2) (at 97.79 265.43 0)
+    (property "Footprint" "lpddr4-test-board-footprints:" (id 2) (at 97.79 265.43 0)
       (effects (font (size 1.27 1.27)) hide)
     )
@@
     )
     (property "Value" "GND" (id 1) (at 123.952 269.1892 0))
-    (property "Footprint" "" (id 2) (at 123.825 264.795 0)
+    (property "Footprint" "lpddr4-test-board-footprints:" (id 2) (at 123.825 264.795 0)
       (effects (font (size 1.27 1.27)) hide)
     )
@@
     )
     (property "Value" "GND" (id 1) (at 217.297 229.8192 0))
-    (property "Footprint" "" (id 2) (at 217.17 225.425 0)
+    (property "Footprint" "lpddr4-test-board-footprints:" (id 2) (at 217.17 225.425 0)
       (effects (font (size 1.27 1.27)) hide)
     )
@@
     )
     (property "Value" "GND" (id 1) (at 44.577 137.7442 0))
-    (property "Footprint" "" (id 2) (at 44.45 133.35 0)
+    (property "Footprint" "lpddr4-test-board-footprints:" (id 2) (at 44.45 133.35 0)
       (effects (font (size 1.27 1.27)) hide)
     )
@@
     )
     (property "Value" "GND" (id 1) (at 73.025 133.9834 0))
-    (property "Footprint" "" (id 2) (at 73.025 129.54 0)
+    (property "Footprint" "lpddr4-test-board-footprints:" (id 2) (at 73.025 129.54 0)
       (effects (font (size 1.27 1.27)) hide)
     )
@@
     )
     (property "Value" "GND" (id 1) (at 110.617 191.0842 0))
-    (property "Footprint" "" (id 2) (at 110.49 186.69 0)
+    (property "Footprint" "lpddr4-test-board-footprints:" (id 2) (at 110.49 186.69 0)
       (effects (font (size 1.27 1.27)) hide)
     )
@@
     )
     (property "Value" "GND" (id 1) (at 90.297 191.0842 0))
-    (property "Footprint" "" (id 2) (at 90.17 186.69 0)
+    (property "Footprint" "lpddr4-test-board-footprints:" (id 2) (at 90.17 186.69 0)
       (effects (font (size 1.27 1.27)) hide)
     )
@@
     )
     (property "Value" "GND" (id 1) (at 82.677 191.0842 0))
-    (property "Footprint" "" (id 2) (at 82.55 186.69 0)
+    (property "Footprint" "lpddr4-test-board-footprints:" (id 2) (at 82.55 186.69 0)
       (effects (font (size 1.27 1.27)) hide)
     )
@@
     )
     (property "Value" "GND" (id 1) (at 62.357 191.0842 0))
-    (property "Footprint" "" (id 2) (at 62.23 186.69 0)
+    (property "Footprint" "lpddr4-test-board-footprints:" (id 2) (at 62.23 186.69 0)
       (effects (font (size 1.27 1.27)) hide)
     )
@@
     )
     (property "Value" "GND" (id 1) (at 44.577 229.8192 0))
-    (property "Footprint" "" (id 2) (at 44.45 225.425 0)
+    (property "Footprint" "lpddr4-test-board-footprints:" (id 2) (at 44.45 225.425 0)
       (effects (font (size 1.27 1.27)) hide)
     )
@@
     )
     (property "Value" "GND" (id 1) (at 52.197 229.8192 0))
-    (property "Footprint" "" (id 2) (at 52.07 225.425 0)
+    (property "Footprint" "lpddr4-test-board-footprints:" (id 2) (at 52.07 225.425 0)
       (effects (font (size 1.27 1.27)) hide)
     )
@@
     )
     (property "Value" "GND" (id 1) (at 59.817 229.8192 0))
-    (property "Footprint" "" (id 2) (at 59.69 225.425 0)
+    (property "Footprint" "lpddr4-test-board-footprints:" (id 2) (at 59.69 225.425 0)
       (effects (font (size 1.27 1.27)) hide)
     )
@@
     )
     (property "Value" "GND" (id 1) (at 67.437 229.8192 0))
-    (property "Footprint" "" (id 2) (at 67.31 225.425 0)
+    (property "Footprint" "lpddr4-test-board-footprints:" (id 2) (at 67.31 225.425 0)
       (effects (font (size 1.27 1.27)) hide)
     )
@@
     )
     (property "Value" "GND" (id 1) (at 56.642 265.3792 0))
-    (property "Footprint" "" (id 2) (at 56.515 260.985 0)
+    (property "Footprint" "lpddr4-test-board-footprints:" (id 2) (at 56.515 260.985 0)
       (effects (font (size 1.27 1.27)) hide)
     )
@@
     )
     (property "Value" "GND" (id 1) (at 64.262 265.3792 0))
-    (property "Footprint" "" (id 2) (at 64.135 260.985 0)
+    (property "Footprint" "lpddr4-test-board-footprints:" (id 2) (at 64.135 260.985 0)
       (effects (font (size 1.27 1.27)) hide)
     )
@@
     )
     (property "Value" "GND" (id 1) (at 49.022 265.3792 0))
-    (property "Footprint" "" (id 2) (at 48.895 260.985 0)
+    (property "Footprint" "lpddr4-test-board-footprints:" (id 2) (at 48.895 260.985 0)
       (effects (font (size 1.27 1.27)) hide)
     )
@@
     )
     (property "Value" "GND" (id 1) (at 226.822 155.5242 0))
-    (property "Footprint" "" (id 2) (at 226.695 151.13 0)
+    (property "Footprint" "lpddr4-test-board-footprints:" (id 2) (at 226.695 151.13 0)
       (effects (font (size 1.27 1.27)) hide)
     )
@@
     )
     (property "Value" "GND" (id 1) (at 239.522 168.2242 0))
-    (property "Footprint" "" (id 2) (at 239.395 163.83 0)
+    (property "Footprint" "lpddr4-test-board-footprints:" (id 2) (at 239.395 163.83 0)
       (effects (font (size 1.27 1.27)) hide)
     )
@@
     )
     (property "Value" "GND" (id 1) (at 203.962 155.5242 0))
-    (property "Footprint" "" (id 2) (at 203.835 151.13 0)
+    (property "Footprint" "lpddr4-test-board-footprints:" (id 2) (at 203.835 151.13 0)
       (effects (font (size 1.27 1.27)) hide)
     )
@@
     )
     (property "Value" "GND" (id 1) (at 254.762 106.6292 0))
-    (property "Footprint" "" (id 2) (at 254.635 102.235 0)
+    (property "Footprint" "lpddr4-test-board-footprints:" (id 2) (at 254.635 102.235 0)
       (effects (font (size 1.27 1.27)) hide)
     )
@@
     )
     (property "Value" "GND" (id 1) (at 260.477 106.6292 0))
-    (property "Footprint" "" (id 2) (at 260.35 102.235 0)
+    (property "Footprint" "lpddr4-test-board-footprints:" (id 2) (at 260.35 102.235 0)
       (effects (font (size 1.27 1.27)) hide)
     )
@@
     )
     (property "Value" "GND" (id 1) (at 280.797 106.6292 0))
-    (property "Footprint" "" (id 2) (at 280.67 102.235 0)
+    (property "Footprint" "lpddr4-test-board-footprints:" (id 2) (at 280.67 102.235 0)
       (effects (font (size 1.27 1.27)) hide)
     )
@@
     )
     (property "Value" "GND" (id 1) (at 339.852 111.7092 0))
-    (property "Footprint" "" (id 2) (at 339.725 107.315 0)
+    (property "Footprint" "lpddr4-test-board-footprints:" (id 2) (at 339.725 107.315 0)
       (effects (font (size 1.27 1.27)) hide)
     )
@@
     )
     (property "Value" "GND" (id 1) (at 337.947 220.9292 0))
-    (property "Footprint" "" (id 2) (at 337.82 216.535 0)
+    (property "Footprint" "lpddr4-test-board-footprints:" (id 2) (at 337.82 216.535 0)
       (effects (font (size 1.27 1.27)) hide)
     )
@@
     )
     (property "Value" "GND" (id 1) (at 73.152 191.0842 0))
-    (property "Footprint" "" (id 2) (at 73.025 186.69 0)
+    (property "Footprint" "lpddr4-test-board-footprints:" (id 2) (at 73.025 186.69 0)
       (effects (font (size 1.27 1.27)) hide)
     )
@@
     )
     (property "Value" "GND" (id 1) (at 76.835 159.385 0))
-    (property "Footprint" "" (id 2) (at 73.025 161.29 0)
+    (property "Footprint" "lpddr4-test-board-footprints:" (id 2) (at 73.025 161.29 0)
       (effects (font (size 1.27 1.27)) hide)
     )
@@
     (pin "1")
   )
-  (symbol (lib_id "antmicroInterfaceControllers:FT4232H-56Q") (at 110.49 130.81 0) (unit 1)
+  (symbol (lib_id "lpddr4-test-board:FT4232H-56Q") (at 110.49 130.81 0) (unit 1)
     (in_bom yes) (on_board yes) (fields_autoplaced)
     (property "Reference" "U4" (id 0) (at 110.49 68.3059 0)
@@
       (effects (font (size 1.524 1.524)))
     )
-    (property "Footprint" "antmicro-footprints:QFN-56-1EP_8x8mm_P0.5mm_EP5.5.9x5.9mm" (id 2) (at 115.57 125.73 90)
+    (property "Footprint" "lpddr4-test-board-footprints:QFN-56-1EP_8x8mm_P0.5mm_EP5.5.9x5.9mm" (id 2) (at 115.57 125.73 90)
       (effects (font (size 1.524 1.524)) (justify left) hide)
     )
@@
     )
     (property "Value" "GND" (id 1) (at 217.297 269.1892 0))
-    (property "Footprint" "" (id 2) (at 217.17 264.795 0)
+    (property "Footprint" "lpddr4-test-board-footprints:" (id 2) (at 217.17 264.795 0)
       (effects (font (size 1.27 1.27)) hide)
     )
@@
     )
     (property "Value" "GND" (id 1) (at 368.427 207.5942 0))
-    (property "Footprint" "" (id 2) (at 368.3 203.2 0)
+    (property "Footprint" "lpddr4-test-board-footprints:" (id 2) (at 368.3 203.2 0)
       (effects (font (size 1.27 1.27)) hide)
     )
@@
     )
     (property "Value" "GND" (id 1) (at 272.542 249.5042 0))
-    (property "Footprint" "" (id 2) (at 272.415 245.11 0)
+    (property "Footprint" "lpddr4-test-board-footprints:" (id 2) (at 272.415 245.11 0)
       (effects (font (size 1.27 1.27)) hide)
     )
@@
     )
     (property "Value" "GND" (id 1) (at 272.542 229.8192 0))
-    (property "Footprint" "" (id 2) (at 272.415 225.425 0)
+    (property "Footprint" "lpddr4-test-board-footprints:" (id 2) (at 272.415 225.425 0)
       (effects (font (size 1.27 1.27)) hide)
     )
@@
     )
     (property "Value" "GND" (id 1) (at 217.932 249.5042 0))
-    (property "Footprint" "" (id 2) (at 217.805 245.11 0)
-      (effects (font (size 1.27 1.27)) hide)
-    )
+    (property "Footprint" "lpddr4-test-board-footprints:" (id 2) (at 217.805 245.11 0)
+      (effects (font (size 1.27 1.27)) hide)
+    )

Commit message: Introduce standardized components
Parts:
- removed J1: WE_629105150521, lpddr4-test-board-footprints:USB_Micro_B_Female_629105150521, symbol lpddr4-test-board:WE_629105150521
- removed J2: 685119134923, lpddr4-test-board-footprints:HDMI_A_Female_685119134923, symbol lpddr4-test-board:685119134923
- added J1: USB-Micro-B_629105150521, antmicro-footprints:USB_Micro_B_Female_629105150521, symbol antmicroUSBDVIHDMIConnectors:USB-Micro-B_629105150521
- added J2: HDMI-A_685119134923, antmicro-footprints:HDMI-A_Wurth_685119134923, symbol antmicroUSBDVIHDMIConnectors:HDMI-A_685119134923
- C10, C14, C18: footprint lpddr4-test-board-footprints:0402-cap -> lpddr4-test-board-footprints:C_0402_1005Metric; Author (none) -> Antmicro; License (none) -> Apache-2.0; Manufacturer MURATA -> Murata
- C11, C12, C13, C15, C17, C19, C8, C9: value C_100n_0402_6V3 -> C_100n_6V3_0402; footprint lpddr4-test-board-footprints:0402-cap -> lpddr4-test-board-footprints:C_0402_1005Metric; symbol lpddr4-test-board:C_100n_0402_6V3 -> lpddr4-test-board:C_100n_6V3_0402; Author (none) -> Antmicro; License (none) -> Apache-2.0
- C16, C20: footprint lpddr4-test-board-footprints:0402-cap -> lpddr4-test-board-footprints:C_0402_1005Metric; Author (none) -> Antmicro; License (none) -> Apache-2.0; Manufacturer MULTICOMP -> Multicomp
- C21: footprint lpddr4-test-board-footprints:0603-cap -> lpddr4-test-board-footprints:C_0603_1608Metric; Author (none) -> Antmicro; License (none) -> Apache-2.0; Manufacturer WALSIN -> Walsin
- D1, D2, D3, D5, D6: value KP-1608CGCK -> LED_G_0603_KP-1608CGCK; footprint lpddr4-test-board-footprints:LED_0603 -> lpddr4-test-board-footprints:LED_0603_1608Metric_G; symbol lpddr4-test-board:KP-1608CGCK -> lpddr4-test-board:LED_G_0603_KP-1608CGCK; Author (none) -> Antmicro; License (none) -> Apache-2.0; Manufacturer KINGBRIGHT -> Kingbright
- D4: value TPD2E009 -> TPD2E009_SOT-9X3; footprint lpddr4-test-board-footprints:SOT-3 -> lpddr4-test-board-footprints:SOT-723; symbol lpddr4-test-board:TPD2E009 -> lpddr4-test-board:TPD2E009_SOT-9X3; Author (none) -> Antmicro; License (none) -> Apache-2.0
- FB1, FB2, FB3: value BLM18AG601SN1D -> FB_600Z_0.5A_0603; footprint lpddr4-test-board-footprints:0603 -> lpddr4-test-board-footprints:FB_0603_1608Metric; symbol lpddr4-test-board:BLM18AG601SN1D -> lpddr4-test-board:FB_600Z_0.5A_0603; Author (none) -> Antmicro; License (none) -> Apache-2.0; Manufacturer Murata Electronics North America -> Murata
- IC1: Author (none) -> Antmicro; License (none) -> Apache-2.0
- J3: value 1140084168 -> MicroSD_1140084168; footprint lpddr4-test-board-footprints:MicroSD_1140084168 -> lpddr4-test-board-footprints:MicroSD_Amphenol_1140084168; symbol lpddr4-test-board:1140084168 -> lpddr4-test-board:MicroSD_1140084168; Author (none) -> Antmicro; License (none) -> Apache-2.0
- Q1, Q2, Q3, Q4, Q5: value BSS138APW -> BSS138PW; symbol lpddr4-test-board:BSS138APW -> lpddr4-test-board:BSS138PW; Author (none) -> Antmicro; License (none) -> Apache-2.0; Manufacturer ON Semiconductor -> Nexperia
- R10, R11, R12, R9: footprint lpddr4-test-board-footprints:0402-res -> lpddr4-test-board-footprints:R_0402_1005Metric; Author (none) -> Antmicro; License (none) -> Apache-2.0; MPN ERJ2GEJ472X -> CR0402-FX-4701GLF; Manufacturer PANASONIC_ELECTRONIC_COMPONENTS -> Bourns; Tolerance (none) -> 1%
- R13, R14, R15, R16, R17, R18, R19, R20, R21, R22, R23, R24, R25: footprint lpddr4-test-board-footprints:0402-res -> lpddr4-test-board-footprints:R_0402_1005Metric; Author (none) -> Antmicro; License (none) -> Apache-2.0; MPN CRCW040222R0FKED -> CR0402-FX-22R0GLF; Manufacturer VISHAY -> Bourns; Tolerance (none) -> 1%
- R26, R27, R28, R29, R30: footprint lpddr4-test-board-footprints:0402-res -> lpddr4-test-board-footprints:R_0402_1005Metric; Author (none) -> Antmicro; License (none) -> Apache-2.0; MPN MCMR04X3300FTL -> CR0402-FX-3300GLF; Manufacturer MULTICOMP -> Bourns; Tolerance (none) -> 1%
- R31, R32, R33, R34, R35, R37, R38: footprint lpddr4-test-board-footprints:0402-res -> lpddr4-test-board-footprints:R_0402_1005Metric; Author (none) -> Antmicro; License (none) -> Apache-2.0; MPN CRCW040220K0FKED -> CR0402-FX-2002GLF; Manufacturer VISHAY -> Bourns; Tolerance (none) -> 1%
- R36: footprint lpddr4-test-board-footprints:0402-res -> lpddr4-test-board-footprints:R_0402_1005Metric; Author (none) -> Antmicro; License (none) -> Apache-2.0; MPN ERJ2GEJ221X -> CR0402-FX-2200GLF; Manufacturer Panasonic -> Bourns; Tolerance (none) -> 1%
- R39, R40, R41, R42, R43, R44, R45, R46: footprint lpddr4-test-board-footprints:0402-res -> lpddr4-test-board-footprints:R_0402_1005Metric; Author (none) -> Antmicro; Current (none) -> 1A; License (none) -> Apache-2.0; Manufacturer PANASONIC -> Panasonic
- R7: footprint lpddr4-test-board-footprints:0402-res -> lpddr4-test-board-footprints:R_0402_1005Metric; Author (none) -> Antmicro; License (none) -> Apache-2.0; MPN CRCW040212K0FKEDHP -> CR0402-FX-1202GLF; Manufacturer VISHAY -> Bourns; Tolerance (none) -> 1%
- R8: footprint lpddr4-test-board-footprints:0402-res -> lpddr4-test-board-footprints:R_0402_1005Metric; Author (none) -> Antmicro; License (none) -> Apache-2.0; MPN CRCW040210K0FKEDHP -> CR0402-FX-1002GLF; Manufacturer VISHAY -> Bourns; Tolerance (none) -> 1%
- TP1, TP2, TP3, TP4, TP5, TP6: value TP_SMD1MM -> TP_1mm_SMD; symbol lpddr4-test-board:TP_SMD1MM -> lpddr4-test-board:TP_1mm_SMD; Author (none) -> Antmicro; License (none) -> Apache-2.0
- U4: value FT4232H-56Q -> FT4232H_VQFN; footprint lpddr4-test-board-footprints:QFN-56-1EP_8x8mm_P0.5mm_EP5.5.9x5.9mm -> lpddr4-test-board-footprints:QFN-56-1EP_8x8mm_P0.5mm; symbol lpddr4-test-board:FT4232H-56Q -> lpddr4-test-board:FT4232H_VQFN; Author (none) -> Antmicro; License (none) -> Apache-2.0
- USR_BTN1, USR_BTN2, USR_BTN3, USR_BTN4: value B3U-1000P -> SW_B3U-1000P; footprint lpddr4-test-board-footprints:Switch_Tactile_SMD_B3U-1000P -> lpddr4-test-board-footprints:SW_B3U-3000P; symbol lpddr4-test-board:B3U-1000P -> lpddr4-test-board:SW_B3U-1000P; Author (none) -> Antmicro; License (none) -> Apache-2.0; Manufacturer Omron Electronics Inc-EMC Div -> Omron Electronics
- Y1: value ABM8G-12.000MHZ-18-D2Y-T -> Oscillator_SMD_12MHz_KX-7; footprint lpddr4-test-board-footprints:KX-7 -> lpddr4-test-board-footprints:Oscillator_SMD_Geyer_KX-7-4Pin_3.2x2.5mm; symbol lpddr4-test-board:ABM8G-12.000MHZ-18-D2Y-T -> lpddr4-test-board:Oscillator_SMD_12MHz_KX-7; Author (none) -> Antmicro; License (none) -> Apache-2.0; Val (none) -> 12MHz
Connections:
- net 1V8_FT: now also C10.2, C13.2, C17.2; no longer C10.1, C13.1, C17.1
- net 3V3_SYS: now also C21.2; no longer C21.1
- net C_TMDS_CLK_N: now also J2.12 (CK-)
- net C_TMDS_CLK_P: now also J2.10 (CK+)
- net C_TMDS_D0_N: now also J2.9 (D0-)
- net C_TMDS_D0_P: now also J2.7 (D0+)
- net C_TMDS_D1_N: now also J2.6 (D1-)
- net C_TMDS_D1_P: now also J2.4 (D1+)
- net C_TMDS_D2_N: now also J2.3 (D2-)
- net C_TMDS_D2_P: now also J2.1 (D2+)
- net DBG_USB_N: now also J1.2 (D-)
- net DBG_USB_P: now also J1.3 (D+)
- net GND: now also C10.1, C11.1, C13.1, C14.1, C16.1, C17.1, C18.1, C20.1, C21.1, C8.1, R7.2, J1.5 (GND), J2.11 (CKS), J2.17 (GND), J2.2 (D2S), J2.5 (D1S), J2.8 (D0S), J2.SH; no longer C10.2, C11.2, C13.2, C14.2, C16.2, C17.2, C18.2, C20.2, C21.2, C8.2, R7.1
- net VBUS: now also J1.1 (VBUS)
- net VPHY: now reaches FB2.2, U4.5 (V_{PHY})
- net VPHY: now also C11.2, C18.2; no longer C11.1, C18.1
- net VPLL: now reaches FB1.2, U4.9 (V_{PLL})
- net VPLL: now also C14.2, C8.2; no longer C14.1, C8.1
- net at U4.6 (REF): now also R7.1; no longer R7.2
- net at U4.3 (OSCI), Y1.1: now also C16.2; no longer C16.1
- net at U4.4 (OSCO), Y1.3: now also C20.2; no longer C20.1
- net at FB3.2: now also J1.SH (SHIELD)
- net at TP2.1: now also J2.13 (CEC)
- net at TP3.1: now also J2.15 (SCL)
- net at TP5.1: now also J2.16 (SDA)
- net at TP6.1: now also J2.18 (+5V)
- net at TP4.1: now also J2.19 (HPD)
- no-connect marks 22 -> 25
Other:
- moved on the sheet: C10, C11, C12, C13, C14, C15, C16, C17, C18, C19, C20, C21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

Commit message: [#55158] components update
Parts:
- J1: footprint antmicro-footprints:USB_Micro_B_Female_629105150521 -> lpddr4-test-board-footprints:USB-Micro-B_Receptacle_WE_629105150521; symbol antmicroUSBDVIHDMIConnectors:USB-Micro-B_629105150521 -> lpddr4-test-board:USB-Micro-B_WE_629105150521
- J2: footprint antmicro-footprints:HDMI-A_Wurth_685119134923 -> lpddr4-test-board-footprints:HDMI-A_Receptacle_WE_685119134923; symbol antmicroUSBDVIHDMIConnectors:HDMI-A_685119134923 -> lpddr4-test-board:HDMI-A_WE_685119134923; Manufacturer Wurth Electronic -> Würth Elektronik
- TP1, TP2, TP3, TP4, TP5, TP6: footprint lpddr4-test-board-footprints:Testpoint_smd_1mm -> antmicro-footprints:TP_SMD_1mm
- U4: Manufacturer FTDI -> FTDI Chip
- USR_BTN1, USR_BTN2, USR_BTN3, USR_BTN4: footprint lpddr4-test-board-footprints:SW_B3U-3000P -> antmicro-footprints:SW_B3U-1000P_SMD; symbol lpddr4-test-board:SW_B3U-1000P -> lpddr4-test-board:SW_B3U-1000P_SMD; Manufacturer Omron Electronics -> Omron
- Y1: symbol lpddr4-test-board:Oscillator_SMD_12MHz_KX-7 -> lpddr4-test-board:Resonator_12MHz_ABM8G; MPN ABM8G-12.000MHZ-18-D2Y-T -> ABM8G-12.000MHZ-18-D2Y-T; Val 12MHz -> 12 MHz
Other:
- moved on the sheet: D4, FB3, IC1, R39, R40, R41, R42, R43, R44, R45, R46, TP2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
